File: hardware/BST900-ESP32/BST900-ESP32.sch (KiCad schematic (older format))
At the start: 14 parts, among them J1 BST900 Left Hand Socket, J2 Thermistor, J3 ADS1115, J4 BST900 Right Hand Socket, U1 TTGO T-DISPLAY

Commit message: New PCB Hardware
Parts:
- removed D1: 3.1V Zener, symbol device:D_Zener
- added C1: 100nF, Capacitor_SMD:C_0805_2012Metric, symbol device:C
- added J3: RS485, Connector_JST:JST_PH_S4B-PH-K_1x04_P2.00mm_Horizontal, symbol conn:Conn_01x04_Male
- added J5: ADS1115, Connector_PinHeader_2.54mm:PinHeader_1x10_P2.54mm_Vertical, symbol Connector:Conn_01x10_Female
- added J7: I2C, Connector_PinHeader_2.54mm:PinHeader_1x04_P2.54mm_Vertical, symbol conn:Conn_01x04_Male
- added JP1: Bus Termination, Jumper:SolderJumper-2_P1.3mm_Open_RoundedPad1.0x1.5mm, symbol Jumper:SolderJumper_2_Open
- added JP2: Power Select, Jumper:SolderJumper-3_P1.3mm_Open_RoundedPad1.0x1.5mm, symbol Jumper:SolderJumper_3_Open
- added R3, R9: 10K, Resistor_SMD:R_0805_2012Metric, symbol device:R
- added R4: 120R, Resistor_SMD:R_0805_2012Metric, symbol device:R
- added R5: 33K, Resistor_SMD:R_0805_2012Metric, symbol device:R
- added R6, R7: 2K2, Resistor_SMD:R_0805_2012Metric, symbol device:R
- added SW1: SW_Push, Button_Switch_SMD:SW_Push_1P1T_NO_6x6mm_H9.5mm, symbol Switch:SW_Push
- added U1: SIT3485ESA, Package_SO:SOIC-8_3.9x4.9mm_P1.27mm, symbol BST900-ESP32:SN65HVD75DR
- C2: renamed from C4; value 470uF -> 470uF 10V; footprint (none) -> Capacitor_SMD:CP_Elec_6.3x7.7; LCSC (none) -> C335982
- C3: renamed from C5; footprint (none) -> Capacitor_SMD:C_0805_2012Metric
- C4: renamed from C1; footprint (none) -> Capacitor_SMD:C_0805_2012Metric
- C5: renamed from C2; footprint (none) -> Capacitor_SMD:C_0805_2012Metric
- C6: renamed from C3; footprint (none) -> Capacitor_SMD:C_0805_2012Metric
- D1: renamed from D2; footprint (none) -> Diode_SMD:D_0805_2012Metric_Pad1.15x1.40mm_HandSolder
- J1: footprint (none) -> Connector_PinHeader_2.54mm:PinHeader_1x08_P2.54mm_Vertical
- J2: footprint (none) -> Connector_PinHeader_2.54mm:PinHeader_1x02_P2.54mm_Horizontal
- J4: renamed from J3; footprint (none) -> Connector_PinHeader_2.54mm:PinHeader_1x10_P2.54mm_Vertical
- J6: renamed from J4; footprint (none) -> Connector_PinHeader_2.54mm:PinHeader_1x08_P2.54mm_Vertical
- R1, R2: footprint (none) -> Resistor_SMD:R_0805_2012Metric
- U2: renamed from U1; footprint (none) -> derek:MODULE_TTGO_T-DISPLAY
Connections:
- net GPIO_36 is gone; now on net ANALOGUE_3: J2.1 (Pin_1), R2.2, U2.23 (Pin_23)
- net CV_CC: no longer D1.2 (A), R1.1, U2.15 (Pin_15)
- net GND: now also C1.2, J3.4 (Pin_4), J5.2 (Pin_2), J7.4 (Pin_4), R5.2, SW1.2, U1.5 (GND)
- net Iout_sense: now also J5.8 (Pin_8), R3.1, R5.1; no longer J1.1 (Pin_1)
- net SCL: now also J5.4 (Pin_4), J7.3 (Pin_3), R6.2
- net SDA: now also J5.3 (Pin_3), J7.2 (Pin_2), R7.2
- net VCC: now also C1.1, J5.1 (Pin_1), J7.1 (Pin_1), R6.1, R7.1, R9.1, U1.8 (VCC); no longer U2.18 (Pin_18)
- net VDD: now also JP2.2 (C); no longer J6.5 (Pin_5), J6.6 (Pin_6)
- net Vin_sense: now also J5.7 (Pin_7)
- net Vout_sense: now also J5.9 (Pin_9)
- net RS485_TX: now reaches U2.16 (Pin_16)
- net RS485_TX: now also U1.4 (D)
- net RS485_RX: now reaches U2.17 (Pin_17)
- net RS485_RX: now also U1.1 (R)
- net GPIO_32: now reaches U2.19 (Pin_19)
- net GPIO_32: now also SW1.1
- net RX485_ENA: now reaches U2.5 (Pin_5)
- net RX485_ENA: now also U1.2 (RE), U1.3 (DE)
- net ANALOGUE_3: now reaches J4.10 (Pin_10)
- net ANALOGUE_3: now also J5.10 (Pin_10)
- net GNDD: no longer names the net of J6.3 (Pin_3), J6.4 (Pin_4)
- new net: J1.1 (Pin_1), R3.2
- new net: J6.5 (Pin_5), J6.6 (Pin_6), JP2.1 (A)
- new net: J3.2 (Pin_2), JP1.2 (B), U1.6 (A)
- new net: J3.3 (Pin_3), R4.1, U1.7 (B)
- new net: JP1.1 (A), R4.2
- new net EXT_5V: J3.1 (Pin_1), JP2.3 (B)
- new net GPIO_27: D1.2 (A), R1.1, U2.15 (Pin_15)
- new net GPIO_33: R9.2, U2.18 (Pin_18)
- no-connect marks 9 -> 6
Other:
- note added: "Accepts both versions of ADS115 modules commonly available on AliExpress.\nThe larger 'Blue' module, or the slimmer 'Purple' module.\nInternal ADC on ESP32 may also be used, but is not recommended."
- note added: "Allows 2.048V range of ADS1115 to be used\n without overflowing at 15A"
- note added: "Blue ADS1115 Module"
- note added: "LED should not be Red. Idea is to use \nforward voltage drop across LED to create a 3.3V safe\ninput for ESP 32. CV_CC pin has 5V on it.\nRed LEDs have too small a forward voltage drop."
- note added: "Not currently used"
- note added: "Note: ver 0.2 had a pot divider on Vout_sense which is not necessary.\nIf using ver 0.2 pcb, Replace resistor with 0R"
- note added: "OR"
- note added: "Pull up resistors on I2c\nNot normally needed since there\nare resistors in the ADS1115 module"
- note added: "Purple ADS1115 Module\n(SDA/SCL reversed)"
- note removed: "Do NOT connect to GND"
- note removed: "Fit either Zener diode OR LED not both.\nLED should not be Red. Idea is to use \nforward voltage drop across LED to create a 3.3V safe\ninput for ESP 32. CV_CC pin has 5V on it.\nRed LEDs have too small a forward voltage drop."
- moved on the sheet: C2, C3, C4, C5, C6, D1, J1, J2, J4, J6, R1, R2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
